Commit message: Update xentrinobot.urdf

File: urdf/xentrinobot.urdf (robot description, URDF)
Before this commit: robot nox, 8 links, 7 joints
Links:
- link base_link: geometry visual mesh filename=package://xentrinobot_101/meshes/base.STL scale=0.001 0.001 0.001
- link kinect: geometry visual mesh filename=package://xentrinobot_101/meshes/kinect_sensor.stl scale=0.01 0.01 0.01
- link motor_left: geometry visual mesh filename=package://xentrinobot_101/meshes/motor.STL scale=0.001 0.001 0.001
- link motor_right: geometry visual mesh filename=package://xentrinobot_101/meshes/motor.STL scale=0.001 0.001 0.001
- link support_wheel_left: geometry visual mesh filename=package://xentrinobot_101/meshes/support_wheel.STL scale=0.001 0.001 0.001
- link support_wheel_right: geometry visual mesh filename=package://xentrinobot_101/meshes/support_wheel.STL scale=0.001 0.001 0.001
- link wheel_left: geometry visual mesh filename=package://xentrinobot_101/meshes/wheel.STL scale=0.001 0.001 0.001
- link wheel_right: geometry visual mesh filename=package://xentrinobot_101/meshes/wheel.STL scale=0.001 0.001 0.001
